File: elec/layout/default/red-llama.kicad_pcb (KiCad board)
At the start: 2 copper layers, 40 x 40 mm, 0 parts

Commit message: fini
Parts:
- added C1: 50V 68nF X7R ±10% 0402 Multilayer Ceramic Capacitors MLCC -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, lib:C0402, F.Cu at (118.0, 85.0)
- added C2: 50V 47pF C0G ±5% 0402 Multilayer Ceramic Capacitors MLCC - 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, lib:C0402, F.Cu at (117.0, 84.0)
- added C3: 16V 33nF X7R ±10% 0402 Multilayer Ceramic Capacitors MLCC -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, lib:C0402, F.Cu at (117.0, 93.0)
- added C4: 50V 100pF C0G ±5% 0402 Multilayer Ceramic Capacitors MLCC -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, lib:C0402, F.Cu at (117.0, 95.5)
- added C5: 10V 10uF X5R ±10% 0603 Multilayer Ceramic Capacitors MLCC -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, lib:C0603, F.Cu at (118.0, 98.0)
- added R1: 125mW Thick Film Resistors 150V ±100ppm/℃ ±1% 1kΩ 0805 Chip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, lib:R0805, F.Cu at (94.1, 85.8)
- added R2: 62.5mW Thick Film Resistors 50V ±100ppm/℃ ±1% 100kΩ 0402 Ch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, lib:R0402, F.Cu at (119.5, 86.3)
- added R3: 62.5mW Thick Film Resistors 50V ±100ppm/℃ ±1% 1MΩ 0402 Chip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, lib:R0402, F.Cu at (120.0, 84.3)
- added R4: 62.5mW Thick Film Resistors 50V ±100ppm/℃ ±1% 100kΩ 0402 Ch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, lib:R0402, F.Cu at (117.5, 88.5)
- added R5: 62.5mW Thick Film Resistors 50V ±100ppm/℃ ±1% 1MΩ 0402 Chip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, lib:R0402, F.Cu at (117.0, 101.0)
- added U1: ?, lib:PDIP-16_L19.7-W6.6-P2.54-LS7.6-BL, F.Cu at (110.7, 91.8)
- added U2: ?, lib:DC-IN-TH_DC-005-5A-2.0-SMT, F.Cu at (91.0, 94.8)
- added U3: ?, lib:CAP-SMD_BD6.3-L6.6-W6.6-LS7.2-R-RD, F.Cu at (100.8, 85.5)
- added U4: ?, lib:SMA_L4.5-W2.7-LS5.1-RD, F.Cu at (100.2, 93.5)
- added U5: ?, lib:HDR-TH_2P-P2.54-V-M-1, F.Cu at (122.0, 85.0)
- added U6: ?, lib:HDR-TH_2P-P2.54-V-M-1, F.Cu at (117.2, 103.0)
- added U7: ?, lib:HDR-TH_2P-P2.54-V-M-1, F.Cu at (89.0, 85.8)
- added U8: ?, lib:HDR-TH_3P-P2.54-V-M-1, F.Cu at (122.0, 92.0)
- added U9: ?, lib:HDR-TH_3P-P2.54-V-M-1, F.Cu at (122.0, 100.5)
Routing:
- net vcc: track 0.00 -> 52.2 mm
- net l_equal_f_hash: track 0.00 -> 20.7 mm
- net gnd: track 0.00 -> 13.6 mm, vias 0 -> 5
- net d: track 0.00 -> 11.7 mm, vias 0 -> 1
- net dc_jack-vcc: track 0.00 -> 9.71 mm
- net j_equal_d_hash: track 0.00 -> 8.54 mm
- net f: track 0.00 -> 7.37 mm
- net output: track 0.00 -> 5.04 mm
- net C6-gnd: track 0.00 -> 4.43 mm
- net p2: track 0.00 -> 4.40 mm
- net input: track 0.00 -> 3.51 mm
- net p1: track 0.00 -> 2.91 mm
- net R2-vcc: track 0.00 -> 1.48 mm
- added copper zone on B.Cu, net gnd
- added copper zone on F.Cu, net gnd
Other:
- board size 40 x 40 mm -> 42 x 24 mm
- board text added: "Hobbs and Lucy December 2024"
- board text added: "RedLLamaWayOverdrive"
